Commit message: limit update

File: hermes_ws/src/my_robot_description/my_robot_description/hermes.urdf (robot description, URDF)
Before this commit: robot my_articulated_robot, 2 links, 3 joints
Joints:
- joint base_to_trailer_pivot: limit (none) -> lower=-3.14159 upper=3.14159 effort=1000.0 velocity=3.0

Commit message: urdf update

File: hermes_ws/src/my_robot_description/my_robot_description/hermes.urdf (robot description, URDF)
Before this commit: robot my_articulated_robot, 2 links, 3 joints
Links:
- removed link trailer_link
- added link fifth_wheel; collision cylinder length=0.05 radius=0.1; visual cylinder length=0.05 radius=0.1
- added link wheel_1; collision cylinder length=0.1 radius=0.05; visual cylinder length=0.1 radius=0.05
- added link wheel_2; collision cylinder length=0.1 radius=0.05; visual cylinder length=0.1 radius=0.05
Joints:
- removed joint base_to_trailer_pivot
- removed joint left_motor_joint
- removed joint right_motor_joint
- added joint base_to_fifth_wheel: type fixed, parent base_link, child fifth_wheel, origin xyz=0 0 0.025 rpy=0 0 0
- added joint fifth_wheel_to_wheel_1: type continuous, parent fifth_wheel, child wheel_1, origin xyz=0 0 0.05 rpy=0 0 0, axis 0 1 0
- added joint fifth_wheel_to_wheel_2: type continuous, parent fifth_wheel, child wheel_2, origin xyz=0 0 -0.05 rpy=0 0 0, axis 0 -1 0

Commit message: urdf file update

File: hermes_ws/src/my_robot_description/my_robot_description/hermes.urdf (robot description, URDF)
Before this commit: robot two_motor_robot, 4 links, 3 joints
Links:
- removed link fifth_wheel
- removed link wheel_1
- removed link wheel_2
- added link fifth_wheel_axle; collision cylinder length=0.05 radius=0.1; visual cylinder length=0.05 radius=0.1
- added link left_motor
- added link right_motor
Joints:
- removed joint base_to_fifth_wheel
- removed joint fifth_wheel_to_wheel_1
- removed joint fifth_wheel_to_wheel_2
- added joint base_to_fifth_wheel_axle: type fixed, parent base_link, child fifth_wheel_axle, origin xyz=0 0 0 rpy=0 0 0
- added joint left_motor_to_fifth_wheel_axle: type continuous, parent left_motor, child fifth_wheel_axle, origin xyz=0 0 0 rpy=0 0 0, axis 1 0 0
- added joint right_motor_to_fifth_wheel_axle: type continuous, parent right_motor, child fifth_wheel_axle, origin xyz=0 0 0 rpy=0 0 0, axis 1 0 0

Commit message: urdf update

File: hermes_ws/src/my_robot_description/my_robot_description/hermes.urdf (robot description, URDF)
Before this commit: robot two_motor_robot, 4 links, 3 joints
Links:
- removed link fifth_wheel_axle
- removed link left_motor
- removed link right_motor
- added link wheel_link; collision cylinder length=0.1 radius=0.05; visual cylinder length=0.1 radius=0.05
- link base_link: geometry collision box size=0.5 0.5 0.1; visual box size=0.5 0.5 0.1
Joints:
- removed joint base_to_fifth_wheel_axle
- removed joint left_motor_to_fifth_wheel_axle
- removed joint right_motor_to_fifth_wheel_axle
- added joint wheel_joint: type revolute, parent base_link, child wheel_link, origin xyz=0 0 0.05 rpy=0 0 0, axis 0 0 1, limit effort=10 velocity=3

Commit message: urdf upd

File: hermes_ws/src/my_robot_description/my_robot_description/hermes.urdf (robot description, URDF)
Before this commit: robot hoverboard, 2 links, 1 joints
Links:
- removed link wheel_link
- added link left_wheel; visual cylinder length=0.05 radius=0.1
- added link right_wheel
- link base_link: geometry visual box size=0.5 0.2 0.1
Joints:
- removed joint wheel_joint
- added joint left_wheel_joint: type continuous, parent base_link, child left_wheel, origin xyz=-0.2 0 0, axis 0 1 0
- added joint right_wheel_joint: type continuous

Commit message: urdf up

File: hermes_ws/src/my_robot_description/my_robot_description/hermes.urdf (robot description, URDF)
Before this commit: robot hoverboard_robot, 3 links, 2 joints
Links:
- link right_wheel: geometry visual cylinder length=0.05 radius=0.1
Joints:
- joint right_wheel_joint: axis (none) -> 0 1 0; child (none) -> right_wheel; origin (none) -> xyz=0.2 0 0; parent (none) -> base_link
