Commit message: urdf file update

File: hermes_ws/src/hermes_urdf/model.urdf (robot description, URDF)
Before this commit: robot onshape, 1 links, 0 joints
Links:
- added link base_link, mass 1.0
- link part_1: mass 1.0 -> None
Joints:
- added joint base_to_part_1: type fixed, parent base_link, child part_1

Commit message: Update model.urdf

File: hermes_ws/src/hermes_urdf/model.urdf (robot description, URDF)
Before this commit: robot onshape, 2 links, 1 joints
Links:
- removed link base_link
- link part_1: mass None -> 1.0; geometry collision mesh filename=file:///home/hermes/Hermes/hermes_ws/src/hermes_urdf/urdf/p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; collision mesh filename=file:///home/hermes/Hermes/hermes_ws/src/hermes_urdf/urdf/r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
Joints:
- removed joint base_to_part_1
