Commit message: urdf code update

File: hermes_ws/src/hermes_urdf/urdf/robot.urdf (robot description, URDF)
Before this commit: robot onshape, 1 links, 0 joints
Links:
- link part_1: mass 0 -> 1.0; geometry collision mesh filename=package://your_package_name/meshes/part_1.stl; collision mesh filename=package://your_package_name/meshes/rehv1.stl

Commit message: urdf file update

File: hermes_ws/src/hermes_urdf/urdf/robot.urdf (robot description, URDF)
Before this commit: robot onshape, 1 links, 0 joints
Links:
- link part_1: geometry collision mesh filename=file:///home/hermes/Hermes/hermes_ws/src/hermes_urdf/urdf/p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; collision mesh filename=file:///home/hermes/Hermes/hermes_ws/src/hermes_urdf/urdf/r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

Commit message: urdf upd

File: hermes_ws/src/hermes_urdf/urdf/robot.urdf (robot description, URDF)
Before this commit: robot onshape, 1 links, 0 joints
Links:
- link part_1: geometry collision mesh filename=file:/home/hermes/Hermes/hermes_ws/src/hermes_urdf/urdf/par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; collision mesh filename=file:/home/hermes/Hermes/hermes_ws/src/hermes_urdf/urdf/reh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

Commit message: urdf update

File: hermes_ws/src/hermes_urdf/urdf/robot.urdf (robot description, URDF)
Before this commit: robot onshape, 1 links, 0 joints
Links:
- added link base_footprint
Joints:
- added joint base_footprint_joint: type fixed, parent base_footprint, child part_1

Commit message: uus urdf file

File: hermes_ws/src/hermes_urdf/urdf/robot.urdf (robot description, URDF)
Before this commit: robot onshape, 2 links, 1 joints
Links:
- removed link base_footprint
- link part_1: mass 1.0 -> 518.58314000823497736; geometry collision mesh filename=package:///ld19.stl; collision mesh filename=package:///part_1.stl
Joints:
- removed joint base_footprint_joint

Commit message: urdf file update

File: hermes_ws/src/hermes_urdf/urdf/robot.urdf (robot description, URDF)
Before this commit: robot onshape, 1 links, 0 joints
Links:
- link part_1: geometry collision mesh filename=file:/home/hermes/Hermes/hermes_ws/src/hermes_urdf/urdf/ld1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; collision mesh filename=file:/home/hermes/Hermes/hermes_ws/src/hermes_urdf/urdf/par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

Commit message: uus urdf file

File: hermes_ws/src/hermes_urdf/urdf/robot.urdf (robot description, URDF)
Before this commit: robot onshape, 1 links, 0 joints
Links:
- added link base_laser, mass 0.1; collision cylinder length=0.1 radius=0.05; visual cylinder length=0.1 radius=0.05
Joints:
- added joint part1_to_base_laser: type fixed, parent part_1, child base_laser, origin xyz=0 0 0 rpy=0 0 0

Commit message: mm

File: hermes_ws/src/hermes_urdf/urdf/robot.urdf (robot description, URDF)
Before this commit: robot onshape, 1 links, 0 joints
Links:
- added link base_laser, mass 0.1; collision box size=0.1 0.1 0.1; visual box size=0.1 0.1 0.1
- added link base_link, mass 1.0; collision box size=1 1 1; visual box size=1 1 1
- link part_1: mass 518.58314000823486367 -> 0
Joints:
- added joint part_1_to_base_laser: type fixed, parent part_1, child base_laser, origin xyz=0.43834751520264569891 -0.10155710888826169347 -0.10871394306610271396 rpy=0 0 -1.570796326794896558
- added joint part_1_to_base_link: type fixed, parent base_link, child part_1, origin xyz=0 0 0 rpy=0 0 0

Commit message: urdf base_link

File: hermes_ws/src/hermes_urdf/urdf/robot.urdf (robot description, URDF)
Before this commit: robot onshape, 3 links, 2 joints
Links:
- removed link base_laser
- removed link part_1
- link base_link: mass 1.0 -> None; geometry visual mesh filename=file:/home/hermes/Hermes/hermes_ws/src/hermes_urdf/urdf/par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
Joints:
- removed joint part_1_to_base_laser
- removed joint part_1_to_base_link
