Commit message: again added ld19 and now added joint

File: hermes_ws/src/hermes_urdf/urdf/hermes.urdf (robot description, URDF)
Before this commit: robot hermes, 1 links, 0 joints
Links:
- added link ld19; visual mesh filename=file:/home/hermes/Hermes/hermes_ws/src/hermes_urdf/urdf/ld1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
Joints:
- added joint base_lidar_joint: type fixed, parent base_link, child ld19, origin xyz=0.43834751520264569891 -0.10155710888826169347 -0.10871394306610271396 rpy=0 -0 -1.570796326794896558

Commit message: changed origin for all

File: hermes_ws/src/hermes_urdf/urdf/hermes.urdf (robot description, URDF)
Before this commit: robot hermes, 2 links, 1 joints
Joints:
- joint base_lidar_joint: origin xyz=0.43834751520264569891 -0.10155710888826169347 -0.10871394306610271396 rpy=0 -0 -1.570796326794896558 -> xyz=0 0 0 rpy=0 0 -1.570796326794896558

Commit message: location change ld19

File: hermes_ws/src/hermes_urdf/urdf/hermes.urdf (robot description, URDF)
Before this commit: robot hermes, 2 links, 1 joints
Joints:
- joint base_lidar_joint: origin xyz=0 0 0 rpy=0 0 -1.570796326794896558 -> xyz=123.0 19.75 42.855 rpy=0 0 -1.570796326794896558

Commit message: measurement reset

File: hermes_ws/src/hermes_urdf/urdf/hermes.urdf (robot description, URDF)
Before this commit: robot hermes, 2 links, 1 joints
Joints:
- joint base_lidar_joint: origin xyz=123.0 19.75 42.855 rpy=0 0 -1.570796326794896558 -> xyz=1.230 0.1975 0.42855 rpy=0 0 -1.570796326794896558

Commit message: location upd ld19

File: hermes_ws/src/hermes_urdf/urdf/hermes.urdf (robot description, URDF)
Before this commit: robot hermes, 2 links, 1 joints
Joints:
- joint base_lidar_joint: origin xyz=1.230 0.1975 0.42855 rpy=0 0 -1.570796326794896558 -> xyz=0.615 0.09875 0.42855 rpy=0 0 0

Commit message: origin upd

File: hermes_ws/src/hermes_urdf/urdf/hermes.urdf (robot description, URDF)
Before this commit: robot hermes, 2 links, 1 joints
Joints:
- joint base_lidar_joint: origin xyz=0.615 0.09875 0.42855 rpy=0 0 0 -> xyz=0.43834751520264569891 -0.10155710888826169347 -0.10871394306610271396 rpy=0 -0 -1.570796326794896558

Commit message: urdf u

File: hermes_ws/src/hermes_urdf/urdf/hermes.urdf (robot description, URDF)
Before this commit: robot hermes, 2 links, 1 joints
Joints:
- joint base_lidar_joint: origin xyz=0.43834751520264569891 -0.10155710888826169347 -0.10871394306610271396 rpy=0 -0 -1.570796326794896558 -> xyz=0.615 0.2775 0.395 rpy=0 0 0

Commit message: loc update

File: hermes_ws/src/hermes_urdf/urdf/hermes.urdf (robot description, URDF)
Before this commit: robot hermes, 2 links, 1 joints
Joints:
- joint base_lidar_joint: origin xyz=0.615 0.2775 0.395 rpy=0 0 0 -> xyz=0.615 0.2775 0.1975 rpy=0 0 0

Commit message: test

File: hermes_ws/src/hermes_urdf/urdf/hermes.urdf (robot description, URDF)
Before this commit: robot hermes, 2 links, 1 joints
Links:
- removed link base_link
- removed link ld19
- added link part_1, mass 0; collision mesh filename=file:/home/hermes/Hermes/hermes_ws/src/hermes_urdf/urdf/ld1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; collision mesh filename=file:/home/hermes/Hermes/hermes_ws/src/hermes_urdf/urdf/par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
Joints:
- removed joint base_lidar_joint

Commit message: test

File: hermes_ws/src/hermes_urdf/urdf/hermes.urdf (robot description, URDF)
Before this commit: robot onshape, 1 links, 0 joints
Links:
- link part_1: geometry visual mesh filename=file:/home/hermes/Hermes/hermes_ws/src/hermes_urdf/urdf/ld1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; visual mesh filename=file:/home/hermes/Hermes/hermes_ws/src/hermes_urdf/urdf/par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

Commit message: kere ratat ld19

File: hermes_ws/src/hermes_urdf/urdf/hermes.urdf (robot description, URDF)
Before this commit: robot onshape, 1 links, 0 joints
Links:
- link part_1: mass 0 -> None; geometry visual mesh filename=file:/home/hermes/Hermes/hermes_ws/src/hermes_urdf/urdf/ld1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; visual mesh filename=file:/home/hermes/Hermes/hermes_ws/src/hermes_urdf/urdf/par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

Commit message: urdf up

File: hermes_ws/src/hermes_urdf/urdf/hermes.urdf (robot description, URDF)
Before this commit: robot onshape, 1 links, 0 joints
Links:
- removed link part_1
- added link base_link; visual mesh filename=file:/home/hermes/Hermes/hermes_ws/src/hermes_urdf/urdf/par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
- added link ld19; visual mesh filename=file:/home/hermes/Hermes/hermes_ws/src/hermes_urdf/urdf/ld1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
Joints:
- added joint base_lidar_joint: type fixed, parent base_link, child ld19, origin xyz=0.43834751520264569891 -0.10155710888826169347 -0.10871394306610271396 rpy=0 -0 -1.570796326794896558

Commit message: no link

File: hermes_ws/src/hermes_urdf/urdf/hermes.urdf (robot description, URDF)
Before this commit: robot hermes, 2 links, 1 joints
Joints:
- removed joint base_lidar_joint

Commit message: test

File: hermes_ws/src/hermes_urdf/urdf/hermes.urdf (robot description, URDF)
Before this commit: robot hermes, 2 links, 0 joints
Joints:
- added joint base_lidar_joint: type fixed, parent base_link, child ld19, origin xyz=0.43834751520264569891 -0.10155710888826169347 -0.10871394306610271396 rpy=0 -0 -1.570796326794896558

Commit message: d

File: hermes_ws/src/hermes_urdf/urdf/hermes.urdf (robot description, URDF)
Before this commit: robot hermes, 2 links, 1 joints
Joints:
- joint base_lidar_joint: origin xyz=0.43834751520264569891 -0.10155710888826169347 -0.10871394306610271396 rpy=0 -0 -1.570796326794896558 -> xyz=0 0 0 rpy=0 -0 -1.570796326794896558

Commit message: joint loc

File: hermes_ws/src/hermes_urdf/urdf/hermes.urdf (robot description, URDF)
Before this commit: robot hermes, 2 links, 1 joints
Joints:
- joint base_lidar_joint: origin xyz=0 0 0 rpy=0 -0 -1.570796326794896558 -> xyz=0.43834751520264569891 -0.10155710888826169347 -0.10871394306610271396 rpy=0 -0 -1.570796326794896558

Commit message: rpy chan

File: hermes_ws/src/hermes_urdf/urdf/hermes.urdf (robot description, URDF)
Before this commit: robot hermes, 2 links, 1 joints
Joints:
- joint base_lidar_joint: origin xyz=0.43834751520264569891 -0.10155710888826169347 -0.10871394306610271396 rpy=0 -0 -1.570796326794896558 -> xyz=0.43834751520264569891 -0.10155710888826169347 -0.10871394306610271396 rpy=0 0 -1.570796326794896558

Commit message: left_front_wheel_update

File: hermes_ws/src/hermes_urdf/urdf/hermes.urdf (robot description, URDF)
Before this commit: robot hermes, 2 links, 1 joints
Links:
- added link front_left_wheel; visual mesh filename=file:/home/hermes/Hermes/hermes_ws/src/hermes_urdf/urdf/reh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
Joints:
- added joint base_front_left_wheel_joint: type continous, parent base_link, child front_left_wheel, origin xyz=-0.65728487905156207649 -0.32390116957514442086 -0.49121394306610272062 rpy=0 -0 0

Commit message: no joint

File: hermes_ws/src/hermes_urdf/urdf/hermes.urdf (robot description, URDF)
Before this commit: robot hermes, 3 links, 2 joints
Joints:
- removed joint base_front_left_wheel_joint

Commit message: no wheel

File: hermes_ws/src/hermes_urdf/urdf/hermes.urdf (robot description, URDF)
Before this commit: robot hermes, 3 links, 1 joints
Links:
- removed link front_left_wheel

Commit message: upd

File: hermes_ws/src/hermes_urdf/urdf/hermes.urdf (robot description, URDF)
Before this commit: robot hermes, 2 links, 1 joints
Links:
- added link front_left_wheel; visual mesh filename=file:/home/hermes/Hermes/hermes_ws/src/hermes_urdf/urdf/reh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
Joints:
- added joint base_front_left_wheel_joint: type fixed, parent base_link, child front_left_wheel, origin xyz=-0.65728487905156207649 -0.32390116957514442086 -0.49121394306610272062 rpy=0 -0 0

Commit message: added axis for wheel

File: hermes_ws/src/hermes_urdf/urdf/hermes.urdf (robot description, URDF)
Before this commit: robot hermes, 3 links, 2 joints
Links:
- removed link front_left_wheel
- added link rear_right_wheel; visual mesh filename=file:/home/hermes/Hermes/hermes_ws/src/hermes_urdf/urdf/reh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
Joints:
- removed joint base_front_left_wheel_joint
- added joint base_rear_wheel_wheel_joint: type fixed, parent base_link, child rear_right_wheel, origin xyz=-0.65728487905156207649 -0.32390116957514442086 -0.49121394306610272062 rpy=0 -0 0, axis 1 0 0

Commit message: rear left

File: hermes_ws/src/hermes_urdf/urdf/hermes.urdf (robot description, URDF)
Before this commit: robot hermes, 3 links, 2 joints
Links:
- added link rear_left_wheel; visual mesh filename=file:/home/hermes/Hermes/hermes_ws/src/hermes_urdf/urdf/reh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
Joints:
- removed joint base_rear_wheel_wheel_joint
- added joint base_rear_left_wheel_joint: type fixed, parent base_link, child rear_left_wheel, origin xyz=0.22271512094843803897 0.17609883042485588445 -0.49121394306610272062 rpy=0 -0 0, axis 1 0 0
- added joint base_rear_right_wheel_joint: type fixed, parent base_link, child rear_right_wheel, origin xyz=-0.65728487905156207649 -0.32390116957514442086 -0.49121394306610272062 rpy=0 -0 0, axis 1 0 0

Commit message: name fix

File: hermes_ws/src/hermes_urdf/urdf/hermes.urdf (robot description, URDF)
Before this commit: robot hermes, 4 links, 3 joints
Links:
- removed link rear_left_wheel
- added link front_left_wheel; visual mesh filename=file:/home/hermes/Hermes/hermes_ws/src/hermes_urdf/urdf/reh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
Joints:
- removed joint base_rear_left_wheel_joint
- added joint base_front_left_wheel_joint: type continuous, parent base_link, child front_left_wheel, origin xyz=0.22271512094843803897 0.17609883042485588445 -0.49121394306610272062 rpy=0 -0 0, axis 1 0 0
- joint base_rear_right_wheel_joint: type fixed -> continuous

Commit message: fixed

File: hermes_ws/src/hermes_urdf/urdf/hermes.urdf (robot description, URDF)
Before this commit: robot hermes, 4 links, 3 joints
Joints:
- joint base_front_left_wheel_joint: type continuous -> fixed
- joint base_rear_right_wheel_joint: type continuous -> fixed

Commit message: removed axis

File: hermes_ws/src/hermes_urdf/urdf/hermes.urdf (robot description, URDF)
Before this commit: robot hermes, 4 links, 3 joints
Joints:
- joint base_front_left_wheel_joint: axis 1 0 0 -> (none)
- joint base_rear_right_wheel_joint: axis 1 0 0 -> (none)

Commit message: fixed to continous

File: hermes_ws/src/hermes_urdf/urdf/hermes.urdf (robot description, URDF)
Before this commit: robot hermes, 4 links, 3 joints
Joints:
- joint base_front_left_wheel_joint: type fixed -> continuous
- joint base_rear_right_wheel_joint: type fixed -> continuous

Commit message: added axis

File: hermes_ws/src/hermes_urdf/urdf/hermes.urdf (robot description, URDF)
Before this commit: robot hermes, 4 links, 3 joints
Joints:
- joint base_front_left_wheel_joint: axis (none) -> 0 1 0
- joint base_rear_right_wheel_joint: axis (none) -> 0 1 0

Commit message: change

File: hermes_ws/src/hermes_urdf/urdf/hermes.urdf (robot description, URDF)
Before this commit: robot hermes, 4 links, 3 joints
Joints:
- joint base_front_left_wheel_joint: origin xyz=0.22271512094843803897 0.17609883042485588445 -0.49121394306610272062 rpy=0 -0 0 -> xyz=0.22271512094843803897 0.17609883042485588445 -0.49121394306610272062 rpy=0 0 0

Commit message: origin

File: hermes_ws/src/hermes_urdf/urdf/hermes.urdf (robot description, URDF)
Before this commit: robot hermes, 4 links, 3 joints
Joints:
- joint base_front_left_wheel_joint: origin xyz=0.22271512094843803897 0.17609883042485588445 -0.49121394306610272062 rpy=0 0 0 -> xyz=0 0 0 rpy=0 0 0

Commit message: .

File: hermes_ws/src/hermes_urdf/urdf/hermes.urdf (robot description, URDF)
Before this commit: robot hermes, 4 links, 3 joints
Links:
- added link rear_left_wheel; visual mesh filename=file:/home/hermes/Hermes/hermes_ws/src/hermes_urdf/urdf/reh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
Joints:
- added joint base_rear_left_wheel_joint: type continuous, parent base_link, child rear_left_wheel, origin xyz=-0.65728487905156196547 0.17609883042485588445 -0.49121394306610272062 rpy=0 0 0, axis 0 1 0

Commit message: .

File: hermes_ws/src/hermes_urdf/urdf/hermes.urdf (robot description, URDF)
Before this commit: robot hermes, 5 links, 4 joints
Joints:
- joint base_rear_left_wheel_joint: type continuous -> fixed

Commit message: .

File: hermes_ws/src/hermes_urdf/urdf/hermes.urdf (robot description, URDF)
Before this commit: robot hermes, 5 links, 4 joints
Links:
- added link front_right_wheel; visual mesh filename=file:/home/hermes/Hermes/hermes_ws/src/hermes_urdf/urdf/reh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
Joints:
- added joint base_front_right_wheel_joint: type fixed, parent base_link, child front_right_wheel, origin xyz=0.22271512094843792795 -0.32390116957514442086 -0.49121394306610272062 rpy=0 0 0, axis 0 1 0

Commit message: d

File: hermes_ws/src/hermes_urdf/urdf/hermes.urdf (robot description, URDF)
Before this commit: robot hermes, 6 links, 5 joints
Links:
- added link base_footprint
Joints:
- added joint base_joint: type fixed, parent base_footprint, child base_link, origin xyz=0 0 0.1 rpy=0 0 0
- joint base_front_right_wheel_joint: axis 0 1 0 -> 1 0 0; type fixed -> continuous
- joint base_rear_left_wheel_joint: type fixed -> continuous
- joint base_rear_right_wheel_joint: axis 0 1 0 -> 1 0 0

Commit message: 0.15

File: hermes_ws/src/hermes_urdf/urdf/hermes.urdf (robot description, URDF)
Before this commit: robot hermes, 7 links, 6 joints
Joints:
- joint base_joint: origin xyz=0 0 0.1 rpy=0 0 0 -> xyz=0 0 0.15 rpy=0 0 0

Commit message: 0.5

File: hermes_ws/src/hermes_urdf/urdf/hermes.urdf (robot description, URDF)
Before this commit: robot hermes, 7 links, 6 joints
Joints:
- joint base_joint: origin xyz=0 0 0.15 rpy=0 0 0 -> xyz=0 0 0.5 rpy=0 0 0

Commit message: 0.15

File: hermes_ws/src/hermes_urdf/urdf/hermes.urdf (robot description, URDF)
Before this commit: robot hermes, 7 links, 6 joints
Joints:
- joint base_joint: origin xyz=0 0 0.5 rpy=0 0 0 -> xyz=0 0 0.15 rpy=0 0 0

Commit message: 0.11

File: hermes_ws/src/hermes_urdf/urdf/hermes.urdf (robot description, URDF)
Before this commit: robot hermes, 7 links, 6 joints
Joints:
- joint base_joint: origin xyz=0 0 0.15 rpy=0 0 0 -> xyz=0 0 0.11 rpy=0 0 0

Commit message: 0.11114

File: hermes_ws/src/hermes_urdf/urdf/hermes.urdf (robot description, URDF)
Before this commit: robot hermes, 7 links, 6 joints
Joints:
- joint base_joint: origin xyz=0 0 0.11 rpy=0 0 0 -> xyz=0 0 0.11114 rpy=0 0 0

Commit message: 02

File: hermes_ws/src/hermes_urdf/urdf/hermes.urdf (robot description, URDF)
Before this commit: robot hermes, 7 links, 6 joints
Joints:
- joint base_joint: origin xyz=0 0 0.11114 rpy=0 0 0 -> xyz=0 0 0.11514 rpy=0 0 0

Commit message: 02

File: hermes_ws/src/hermes_urdf/urdf/hermes.urdf (robot description, URDF)
Before this commit: robot hermes, 7 links, 6 joints
Joints:
- joint base_joint: origin xyz=0 0 0.11514 rpy=0 0 0 -> xyz=0 0 0.12514 rpy=0 0 0

Commit message: 01

File: hermes_ws/src/hermes_urdf/urdf/hermes.urdf (robot description, URDF)
Before this commit: robot hermes, 7 links, 6 joints
Joints:
- joint base_joint: origin xyz=0 0 0.12514 rpy=0 0 0 -> xyz=0 0 0.13514 rpy=0 0 0

Commit message: 1

File: hermes_ws/src/hermes_urdf/urdf/hermes.urdf (robot description, URDF)
Before this commit: robot hermes, 7 links, 6 joints
Joints:
- joint base_joint: origin xyz=0 0 0.13514 rpy=0 0 0 -> xyz=0 0 1.13514 rpy=0 0 0

Commit message: 05

File: hermes_ws/src/hermes_urdf/urdf/hermes.urdf (robot description, URDF)
Before this commit: robot hermes, 7 links, 6 joints
Joints:
- joint base_joint: origin xyz=0 0 1.13514 rpy=0 0 0 -> xyz=0 0 0.53514 rpy=0 0 0

Commit message: removed base

File: hermes_ws/src/hermes_urdf/urdf/hermes.urdf (robot description, URDF)
Before this commit: robot hermes, 7 links, 6 joints
Joints:
- removed joint base_joint

Commit message: removed most of the model

File: hermes_ws/src/hermes_urdf/urdf/hermes.urdf (robot description, URDF)
Before this commit: robot hermes, 7 links, 5 joints
Links:
- removed link front_left_wheel
- removed link front_right_wheel
- removed link ld19
- removed link rear_left_wheel
- removed link rear_right_wheel
Joints:
- removed joint base_front_left_wheel_joint
- removed joint base_front_right_wheel_joint
- removed joint base_lidar_joint
- removed joint base_rear_left_wheel_joint
- removed joint base_rear_right_wheel_joint

Commit message: most of the model is back

File: hermes_ws/src/hermes_urdf/urdf/hermes.urdf (robot description, URDF)
Before this commit: robot hermes, 2 links, 0 joints
Links:
- added link front_left_wheel; visual mesh filename=file:/home/hermes/Hermes/hermes_ws/src/hermes_urdf/urdf/reh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
- added link front_right_wheel; visual mesh filename=file:/home/hermes/Hermes/hermes_ws/src/hermes_urdf/urdf/reh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
- added link ld19; visual mesh filename=file:/home/hermes/Hermes/hermes_ws/src/hermes_urdf/urdf/ld1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
- added link rear_left_wheel; visual mesh filename=file:/home/hermes/Hermes/hermes_ws/src/hermes_urdf/urdf/reh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
- added link rear_right_wheel; visual mesh filename=file:/home/hermes/Hermes/hermes_ws/src/hermes_urdf/urdf/reh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
Joints:
- added joint base_front_left_wheel_joint: type continuous, parent base_link, child front_left_wheel, origin xyz=0.22271512094843803897 0.17609883042485588445 -0.49121394306610272062 rpy=0 0 0, axis 0 1 0
- added joint base_front_right_wheel_joint: type continuous, parent base_link, child front_right_wheel, origin xyz=0.22271512094843792795 -0.32390116957514442086 -0.49121394306610272062 rpy=0 0 0, axis 1 0 0
- added joint base_joint: type fixed, parent base_footprint, child base_link, origin xyz=0 0 0.53514 rpy=0 0 0
- added joint base_lidar_joint: type fixed, parent base_link, child ld19, origin xyz=0.43834751520264569891 -0.10155710888826169347 -0.10871394306610271396 rpy=0 0 -1.570796326794896558
- added joint base_rear_left_wheel_joint: type continuous, parent base_link, child rear_left_wheel, origin xyz=-0.65728487905156196547 0.17609883042485588445 -0.49121394306610272062 rpy=0 0 0, axis 0 1 0
- added joint base_rear_right_wheel_joint: type continuous, parent base_link, child rear_right_wheel, origin xyz=-0.65728487905156207649 -0.32390116957514442086 -0.49121394306610272062 rpy=0 -0 0, axis 1 0 0

Commit message: cont to fixed

File: hermes_ws/src/hermes_urdf/urdf/hermes.urdf (robot description, URDF)
Before this commit: robot hermes, 7 links, 6 joints
Joints:
- joint base_front_left_wheel_joint: type continuous -> fixed
- joint base_front_right_wheel_joint: type continuous -> fixed
- joint base_rear_left_wheel_joint: type continuous -> fixed
- joint base_rear_right_wheel_joint: type continuous -> fixed

Commit message: back to cont

File: hermes_ws/src/hermes_urdf/urdf/hermes.urdf (robot description, URDF)
Before this commit: robot hermes, 7 links, 6 joints
Joints:
- joint base_front_left_wheel_joint: type fixed -> continuous
- joint base_front_right_wheel_joint: type fixed -> continuous
- joint base_rear_left_wheel_joint: type fixed -> continuous
- joint base_rear_right_wheel_joint: type fixed -> continuous

Commit message: base_foorprint update

File: hermes_ws/src/hermes_urdf/urdf/hermes.urdf (robot description, URDF)
Before this commit: robot hermes, 7 links, 6 joints
Joints:
- joint base_joint: origin xyz=0 0 0.53514 rpy=0 0 0 -> xyz=0 0 0.61514 rpy=0 0 0

Commit message: heigh update

File: hermes_ws/src/hermes_urdf/urdf/hermes.urdf (robot description, URDF)
Before this commit: robot hermes, 7 links, 6 joints
Joints:
- joint base_joint: origin xyz=0 0 0.61514 rpy=0 0 0 -> xyz=0 0 0.8514 rpy=0 0 0

Commit message: hieght upd

File: hermes_ws/src/hermes_urdf/urdf/hermes.urdf (robot description, URDF)
Before this commit: robot hermes, 7 links, 6 joints
Joints:
- joint base_joint: origin xyz=0 0 0.8514 rpy=0 0 0 -> xyz=0 0 0.0 rpy=0 0 0

Commit message: height upd

File: hermes_ws/src/hermes_urdf/urdf/hermes.urdf (robot description, URDF)
Before this commit: robot hermes, 7 links, 6 joints
Joints:
- joint base_joint: origin xyz=0 0 0.0 rpy=0 0 0 -> xyz=0 0.5 0.0 rpy=0 0 0

Commit message: height u

File: hermes_ws/src/hermes_urdf/urdf/hermes.urdf (robot description, URDF)
Before this commit: robot hermes, 7 links, 6 joints
Joints:
- joint base_joint: origin xyz=0 0.5 0.0 rpy=0 0 0 -> xyz=0.5 0.0 0.0 rpy=0 0 0

Commit message: test upd heigh

File: hermes_ws/src/hermes_urdf/urdf/hermes.urdf (robot description, URDF)
Before this commit: robot hermes, 7 links, 6 joints
Joints:
- joint base_joint: origin xyz=0.5 0.0 0.0 rpy=0 0 0 -> xyz=1 1 1 rpy=0 0 0

Commit message: test

File: hermes_ws/src/hermes_urdf/urdf/hermes.urdf (robot description, URDF)
Before this commit: robot hermes, 7 links, 6 joints
Joints:
- joint base_joint: origin xyz=1 1 1 rpy=0 0 0 -> xyz=50 50 50 rpy=0 0 0

Commit message: ?

File: hermes_ws/src/hermes_urdf/urdf/hermes.urdf (robot description, URDF)
Before this commit: robot hermes, 7 links, 6 joints
Joints:
- joint base_joint: origin xyz=50 50 50 rpy=0 0 0 -> xyz=50 50 50 rpy=1 1 1

Commit message: updated height

File: hermes_ws/src/hermes_urdf/urdf/hermes.urdf (robot description, URDF)
Before this commit: robot hermes, 7 links, 6 joints
Joints:
- joint base_joint: origin xyz=50 50 50 rpy=1 1 1 -> xyz=0 0 0.7 rpy=0 0 0

Commit message: uus urdf file

File: hermes_ws/src/hermes_urdf/urdf/hermes.urdf (robot description, URDF)
Before this commit: robot hermes, 7 links, 6 joints
Links:
- added link liigend; visual mesh filename=file:/home/hermes/Hermes/hermes_ws/src/hermes_urdf/urdf/lii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
- link base_link: geometry visual mesh filename=file:/home/hermes/Hermes/hermes_ws/src/hermes_urdf/urdf/ker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
Joints:
- added joint liigend_to_kere_joint: type continuous, parent base_link, child liigend, origin xyz=0.9483341292917655263 -0.0071774303769965852595 0.6075567520903586427 rpy=2.2686993105948162011e-15 -6.1350116673315255536e-22 -1.5707963267948390484, axis 0 0 1
- joint base_front_left_wheel_joint: origin xyz=0.22271512094843803897 0.17609883042485588445 -0.49121394306610272062 rpy=0 0 0 -> xyz=0.9483341292917480958 0.29532256962300351688 0.60755675209035853168 rpy=-5.7841602488177229343e-14 1.5707963267948958919 0
- joint base_front_right_wheel_joint: origin xyz=0.22271512094843792795 -0.32390116957514442086 -0.49121394306610272062 rpy=0 0 0 -> xyz=0.9483341292917799592 -0.2596774303769966985 0.6075567520903586427 rpy=-6.1350056294378907142e-22 -2.2686993105950812583e-15 5.7620574978045523474e-14
- joint base_lidar_joint: origin xyz=0.43834751520264569891 -0.10155710888826169347 -0.10871394306610271396 rpy=0 0 -1.570796326794896558 -> xyz=1.039666598485702087 -0.0073333696901138160917 0.99755675209036465123 rpy=1.4644253098708029941e-15 7.9409344339936499792e-23 -1.5707963267948970021
- joint base_rear_left_wheel_joint: origin xyz=-0.65728487905156196547 0.17609883042485588445 -0.49121394306610272062 rpy=0 0 0 -> xyz=0.06653420423147499152 0.25032256962300086789 0.61255675209034965434 rpy=3.141592653589793116 1.8665624601511276584e-15 -3.1415926535897926719
- joint base_rear_right_wheel_joint: origin xyz=-0.65728487905156207649 -0.32390116957514442086 -0.49121394306610272062 rpy=0 -0 0 -> xyz=0.066534204231474658453 -0.26467743037699664743 0.61255675209034976536 rpy=7.940934590483602961e-23 -1.4644253098708242934e-15 1.55431223447518563e-15
