Commit message: d

File: hermes_ws/src/hermes_urdf/urdf/hermes.urdf (robot description, URDF)
Before this commit: robot hermes, 8 links, 7 joints
Joints:
- joint base_rear_right_wheel_joint: origin xyz=0.066534204231474658453 -0.26467743037699664743 0.61255675209034976536 rpy=7.940934590483602961e-23 -1.4644253098708242934e-15 1.55431223447518563e-15 -> xyz=0.066534204231474658453 -0.21467743037699693609 0.61255675209034976536 rpy=3.3611923249190478047e-30 -1.8665624601511304194e-15 5.6898930012037971076e-16
