Commit message: launch file update

File: hermes_ws/src/hermes_urdf/urdf/hermes_model.urdf (robot description, URDF)
Before this commit: robot hermes, 8 links, 7 joints
Links:
- link base_link: geometry visual mesh filename=file:/home/hermes/Hermes/hermes_ws/src/hermes_urdf/urdf/ker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
- link front_left_wheel: geometry visual mesh filename=file:/home/hermes/Hermes/hermes_ws/src/hermes_urdf/urdf/reh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
- link front_right_wheel: geometry visual mesh filename=file:/home/hermes/Hermes/hermes_ws/src/hermes_urdf/urdf/reh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
- link ld19: geometry visual mesh filename=file:/home/hermes/Hermes/hermes_ws/src/hermes_urdf/urdf/ld1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
- link rear_left_wheel: geometry visual mesh filename=file:/home/hermes/Hermes/hermes_ws/src/hermes_urdf/urdf/reh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
- link rear_right_wheel: geometry visual mesh filename=file:/home/hermes/Hermes/hermes_ws/src/hermes_urdf/urdf/reh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

Commit message: Nav2 libs not working

File: hermes_ws/src/hermes_urdf/urdf/hermes_model.urdf (robot description, URDF)
Before this commit: robot hermes, 8 links, 7 joints
Links:
- added link gps_link; collision box size=0.1 0.1 0.1
Joints:
- added joint gps_joint: type fixed, parent base_link, child gps_link, origin xyz=1.039666598485702087 -0.0073333696901138160917 0.99755675209036465123 rpy=0 0 0

Commit message: uus nav file

File: hermes_ws/src/hermes_urdf/urdf/hermes_model.urdf (robot description, URDF)
Before this commit: robot hermes, 9 links, 8 joints
Links:
- added link ld19, mass 2.0; visual mesh filename=/home/aleksmalm/Hermes/hermes_ws/src/hermes_urdf/urdf/ld19.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
Joints:
- added joint base_lidar_joint: type fixed, parent base_link, child ld19, origin xyz=1.039666598485702087 -0.0073333696901138160917 0.99755675209036465123 rpy=1.4644253098708029941e-15 7.9409344339936499792e-23 -1.5707963267948970021

Commit message: uus urdf ja nav

File: hermes_ws/src/hermes_urdf/urdf/hermes_model.urdf (robot description, URDF)
Before this commit: robot hermes, 10 links, 9 joints
Links:
- removed link base_link_front
- removed link gps_link
- added link imu_link
- link base_link: mass 50.0 -> 25.0; geometry collision mesh filename=package://hermes_urdf/urdf/kere.stl; visual mesh filename=package://hermes_urdf/urdf/kere.stl
- link front_left_wheel: mass 1.5 -> 10.0; geometry collision mesh filename=package://hermes_urdf/urdf/rehv.stl; visual mesh filename=package://hermes_urdf/urdf/rehv.stl
- link front_right_wheel: mass 1.5 -> 10.0; geometry collision mesh filename=package://hermes_urdf/urdf/rehv.stl; visual mesh filename=package://hermes_urdf/urdf/rehv.stl
- link ld19: mass 2.0 -> 0.1; geometry visual mesh filename=package://hermes_urdf/urdf/ld19.stl
- link liigend: mass 3.0 -> 2.0; geometry visual mesh filename=package://hermes_urdf/urdf/liigend.stl
- link rear_left_wheel: mass 1.5 -> 3.0; geometry collision mesh filename=package://hermes_urdf/urdf/rehv_tagumine.stl; visual mesh filename=package://hermes_urdf/urdf/rehv_tagumine.stl
- link rear_right_wheel: mass 1.5 -> 3.0; geometry collision mesh filename=package://hermes_urdf/urdf/rehv_tagumine.stl; visual mesh filename=package://hermes_urdf/urdf/rehv_tagumine.stl
Joints:
- removed joint base_link_to_front
- removed joint gps_joint
- added joint base_link_to_imu: type fixed, parent base_link, child imu_link, origin xyz=-0.00032976124091513292491 -0.091578898488961058 0.3865718126789312592 rpy=6.3108872417680804303e-30 -2.9537602700216738211e-30 -3.141592653589793116
- joint liigend_to_kere_joint: limit lower=-0.7854 upper=0.7854 effort=100000 velocity=100 -> lower=-0.7854 upper=0.7854 effort=50 velocity=2
