Commit message: urdf file and launch file upd

File: hermes_ws/install/hermes_urdf/share/hermes_urdf/urdf/hermes.urdf (robot description, URDF)
Before this commit: robot hermes, 7 links, 6 joints
Joints:
- joint base_front_left_wheel_joint: type fixed -> continuous
- joint base_front_right_wheel_joint: axis 1 0 0 -> 0 1 0; type fixed -> continuous
- joint base_joint: origin xyz=0 0 0.53514 rpy=0 0 0 -> xyz=0 0 0.61 rpy=0 0 0
- joint base_rear_left_wheel_joint: type fixed -> continuous
- joint base_rear_right_wheel_joint: axis 1 0 0 -> 0 1 0; type fixed -> continuous

File: hermes_ws/src/hermes_urdf/urdf/hermes.urdf (robot description, URDF)
Before this commit: robot hermes, 7 links, 6 joints
Joints:
- joint base_front_right_wheel_joint: axis 1 0 0 -> 0 1 0
- joint base_joint: origin xyz=0 0 0.7 rpy=0 0 0 -> xyz=0 0 0.615 rpy=0 0 0
- joint base_rear_right_wheel_joint: axis 1 0 0 -> 0 1 0

Commit message: d

File: hermes_ws/install/hermes_urdf/share/hermes_urdf/urdf/hermes.urdf (robot description, URDF)
Before this commit: robot hermes, 7 links, 6 joints
Links:
- added link liigend; visual mesh filename=file:/home/hermes/Hermes/hermes_ws/src/hermes_urdf/urdf/lii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
- link base_link: geometry visual mesh filename=file:/home/hermes/Hermes/hermes_ws/src/hermes_urdf/urdf/ker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
Joints:
- added joint liigend_to_kere_joint: type continuous, parent base_link, child liigend, origin xyz=0.9483341292917655263 -0.0071774303769965852595 0.6075567520903586427 rpy=2.2686993105948162011e-15 -6.1350116673315255536e-22 -1.5707963267948390484, axis 0 0 1
- joint base_front_left_wheel_joint: origin xyz=0.22271512094843803897 0.17609883042485588445 -0.49121394306610272062 rpy=0 0 0 -> xyz=0.9483341292917480958 0.29532256962300351688 0.60755675209035853168 rpy=-5.7841602488177229343e-14 1.5707963267948958919 0; parent base_link -> liigend
- joint base_front_right_wheel_joint: origin xyz=0.22271512094843792795 -0.32390116957514442086 -0.49121394306610272062 rpy=0 0 0 -> xyz=0.9483341292917799592 -0.2596774303769966985 0.6075567520903586427 rpy=-6.1350056294378907142e-22 -2.2686993105950812583e-15 5.7620574978045523474e-14; parent base_link -> liigend
- joint base_joint: origin xyz=0 0 0.61 rpy=0 0 0 -> xyz=0 0 0 rpy=0 0 0
- joint base_lidar_joint: origin xyz=0.43834751520264569891 -0.10155710888826169347 -0.10871394306610271396 rpy=0 0 -1.570796326794896558 -> xyz=1.039666598485702087 -0.0073333696901138160917 0.99755675209036465123 rpy=1.4644253098708029941e-15 7.9409344339936499792e-23 -1.5707963267948970021
- joint base_rear_left_wheel_joint: origin xyz=-0.65728487905156196547 0.17609883042485588445 -0.49121394306610272062 rpy=0 0 0 -> xyz=0.06653420423147499152 0.25032256962300086789 0.61255675209034965434 rpy=3.141592653589793116 1.8665624601511276584e-15 -3.1415926535897926719
- joint base_rear_right_wheel_joint: origin xyz=-0.65728487905156207649 -0.32390116957514442086 -0.49121394306610272062 rpy=0 -0 0 -> xyz=0.066534204231474658453 -0.26467743037699664743 0.61255675209034976536 rpy=7.940934590483602961e-23 -1.4644253098708242934e-15 1.55431223447518563e-15

File: hermes_ws/src/hermes_urdf/urdf/hermes.urdf (robot description, URDF)
Before this commit: robot hermes, 8 links, 7 joints
Joints:
- joint base_front_left_wheel_joint: parent base_link -> liigend
- joint base_front_right_wheel_joint: parent base_link -> liigend
- joint base_joint: origin xyz=0 0 0.615 rpy=0 0 0 -> xyz=0 0 0 rpy=0 0 0
