Commit message: new model

File: hermes_ws/install/hermes_urdf/share/hermes_urdf/urdf/hermes_model.urdf (robot description, URDF)
Before this commit: robot hermes, 8 links, 7 joints
Joints:
- joint base_front_left_wheel_joint: axis 0 0 1 -> 1 0 0
- joint base_front_right_wheel_joint: axis 0 0 1 -> 1 0 0

Commit message: s

File: hermes_ws/install/hermes_urdf/share/hermes_urdf/urdf/hermes_model.urdf (robot description, URDF)
Before this commit: robot hermes, 8 links, 7 joints
Links:
- link base_footprint: mass None -> 1.0
- link base_link: mass None -> 5.0; geometry visual mesh filename=/home/hermes/Hermes/hermes_ws/src/hermes_urdf/urdf/kere.stl
- link front_left_wheel: mass None -> 1.5; geometry visual mesh filename=/home/hermes/Hermes/hermes_ws/src/hermes_urdf/urdf/rehv.stl
- link front_right_wheel: mass None -> 1.5; geometry visual mesh filename=/home/hermes/Hermes/hermes_ws/src/hermes_urdf/urdf/rehv.stl
- link ld19: mass None -> 2.0; geometry visual mesh filename=/home/hermes/Hermes/hermes_ws/src/hermes_urdf/urdf/ld19.stl
- link liigend: mass None -> 3.0; geometry visual mesh filename=/home/hermes/Hermes/hermes_ws/src/hermes_urdf/urdf/liigend.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
- link rear_left_wheel: mass None -> 1.5; geometry visual mesh filename=/home/hermes/Hermes/hermes_ws/src/hermes_urdf/urdf/rehv.stl
- link rear_right_wheel: mass None -> 1.5; geometry visual mesh filename=/home/hermes/Hermes/hermes_ws/src/hermes_urdf/urdf/rehv.stl
Joints:
- joint base_joint: origin xyz=0 0 0 rpy=0 0 0 -> xyz=0 0 -0.48 rpy=0 0 0

Commit message: d

File: hermes_ws/install/hermes_urdf/share/hermes_urdf/urdf/hermes_model.urdf (robot description, URDF)
Before this commit: robot hermes, 8 links, 7 joints
Links:
- link base_link: geometry visual mesh filename=file:/home/hermes/Hermes/hermes_ws/src/hermes_urdf/urdf/ker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
- link front_left_wheel: geometry visual mesh filename=file:/home/hermes/Hermes/hermes_ws/src/hermes_urdf/urdf/reh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
- link front_right_wheel: geometry visual mesh filename=file:/home/hermes/Hermes/hermes_ws/src/hermes_urdf/urdf/reh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
- link ld19: geometry visual mesh filename=file:/home/hermes/Hermes/hermes_ws/src/hermes_urdf/urdf/ld1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
- link liigend: geometry visual mesh filename=file:/home/hermes/Hermes/hermes_ws/src/hermes_urdf/urdf/lii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
- link rear_left_wheel: geometry visual mesh filename=file:/home/hermes/Hermes/hermes_ws/src/hermes_urdf/urdf/reh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
- link rear_right_wheel: geometry visual mesh filename=file:/home/hermes/Hermes/hermes_ws/src/hermes_urdf/urdf/reh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

File: hermes_ws/src/hermes_urdf/urdf/hermes_model.urdf (robot description, URDF)
Before this commit: robot hermes, 8 links, 7 joints
Links:
- link liigend: geometry visual mesh filename=file:/home/hermes/Hermes/hermes_ws/src/hermes_urdf/urdf/lii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

Commit message: c

File: hermes_ws/install/hermes_urdf/share/hermes_urdf/urdf/hermes_model.urdf (robot description, URDF)
Before this commit: robot hermes, 8 links, 7 joints
Links:
- link base_link: geometry visual mesh filename=/home/aleksmalm/Hermes/hermes_ws/src/hermes_urdf/urdf/kere.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
- link front_left_wheel: geometry visual mesh filename=/home/aleksmalm/Hermes/hermes_ws/src/hermes_urdf/urdf/rehv.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
- link front_right_wheel: geometry visual mesh filename=/home/aleksmalm/Hermes/hermes_ws/src/hermes_urdf/urdf/rehv.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
- link ld19: geometry visual mesh filename=/home/aleksmalm/Hermes/hermes_ws/src/hermes_urdf/urdf/ld19.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
- link liigend: geometry visual mesh filename=/home/aleksmalm/Hermes/hermes_ws/src/hermes_urdf/urdf/liige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
- link rear_left_wheel: geometry visual mesh filename=/home/aleksmalm/Hermes/hermes_ws/src/hermes_urdf/urdf/rehv.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
- link rear_right_wheel: geometry visual mesh filename=/home/aleksmalm/Hermes/hermes_ws/src/hermes_urdf/urdf/rehv.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

Commit message: update

File: hermes_ws/install/hermes_urdf/share/hermes_urdf/urdf/hermes_model.urdf (robot description, URDF)
Before this commit: robot hermes, 8 links, 7 joints
Links:
- link base_link: geometry collision mesh filename=/home/aleksmalm/Hermes/hermes_ws/src/hermes_urdf/urdf/kere.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; visual mesh filename=/home/aleksmalm/Hermes/hermes_ws/src/hermes_urdf/urdf/kere.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
- link front_left_wheel: geometry collision mesh filename=/home/aleksmalm/Hermes/hermes_ws/src/hermes_urdf/urdf/rehv.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; visual mesh filename=/home/aleksmalm/Hermes/hermes_ws/src/hermes_urdf/urdf/rehv.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
- link front_right_wheel: geometry collision mesh filename=/home/aleksmalm/Hermes/hermes_ws/src/hermes_urdf/urdf/rehv.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; visual mesh filename=/home/aleksmalm/Hermes/hermes_ws/src/hermes_urdf/urdf/rehv.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
- link rear_left_wheel: geometry collision mesh filename=/home/aleksmalm/Hermes/hermes_ws/src/hermes_urdf/urdf/rehv.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; visual mesh filename=/home/aleksmalm/Hermes/hermes_ws/src/hermes_urdf/urdf/rehv.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
- link rear_right_wheel: geometry collision mesh filename=/home/aleksmalm/Hermes/hermes_ws/src/hermes_urdf/urdf/rehv.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; visual mesh filename=/home/aleksmalm/Hermes/hermes_ws/src/hermes_urdf/urdf/rehv.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
Joints:
- joint base_joint: origin xyz=0 0 -0.48 rpy=0 0 0 -> xyz=0 0 -0.45 rpy=0 0 0
- joint liigend_to_kere_joint: limit (none) -> lower=-0.7854 upper=0.7854 effort=100000 velocity=100

Commit message: Uus mudel ilma fyysikata

File: hermes_ws/install/hermes_urdf/share/hermes_urdf/urdf/hermes_model.urdf (robot description, URDF)
Before this commit: robot hermes, 10 links, 9 joints
Links:
- link base_link: mass 5.0 -> 50.0
- link rear_left_wheel: geometry collision mesh filename=/home/aleksmalm/Hermes/hermes_ws/src/hermes_urdf/urdf/rehv_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; visual mesh filename=/home/aleksmalm/Hermes/hermes_ws/src/hermes_urdf/urdf/rehv_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
- link rear_right_wheel: geometry collision mesh filename=/home/aleksmalm/Hermes/hermes_ws/src/hermes_urdf/urdf/rehv_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; visual mesh filename=/home/aleksmalm/Hermes/hermes_ws/src/hermes_urdf/urdf/rehv_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
Joints:
- joint base_front_left_wheel_joint: axis -1 0 0 ->  -1 0 0; origin xyz=-0.30232256962300351688 0 0 rpy=0 0 0 -> xyz=0.30257617807220232864 -0.00024642929502571853106 -0.0034281873210687194287 rpy=0 -0 3.141592653589793116
- joint base_front_right_wheel_joint: origin xyz=0.2523774303769966985 0 0 rpy=0 0 0 -> xyz=-0.30292382192779770955 -0.00024642929502571853106 -0.0034281873210687333065 rpy=0 -0 0
- joint base_joint: origin xyz=0.95 -0.02 -0.46 rpy=0 0 3.14159265359 -> xyz=0 0 0.1 rpy=0 0 0
- joint base_lidar_joint: origin xyz=1.039666598485702087 -0.0073333696901138160917 0.99755675209036465123 rpy=1.4644253098708029941e-15 7.9409344339936499792e-23 -1.5707963267948970021 -> xyz=-0.00032976124091513292491 -0.091578898488961058 0.3865718126789312592 rpy=6.3108872417680804303e-30 -2.9537602700216738211e-30 -3.141592653589793116
- joint base_link_to_front: origin xyz=1.0 0 0 rpy=0 0 0 -> xyz=0 0 0 rpy=0 0 0
- joint base_rear_left_wheel_joint: origin xyz=0.06653420423147499152 0.25032256962300086789 0.61255675209034965434 rpy=3.141592653589793116 1.8665624601511276584e-15 -3.1415926535897926719 -> xyz=-0.207673821927797847 0.88155349576524655308 0.0015718126789312503178 rpy=1.570796326794896558 1.570796326794896558 0
- joint base_rear_right_wheel_joint: origin xyz=0.066534204231474658453 -0.21467743037699693609 0.61255675209034976536 rpy=3.3611923249190478047e-30 -1.8665624601511304194e-15 5.6898930012037971076e-16 -> xyz=0.25732617807220242723 0.88155349576524644206 0.0015718126789312780733 rpy=1.570796326794896558 1.570796326794896558 0
- joint gps_joint: origin xyz=1.0 0 0 rpy=0 0 0 -> xyz=-0.00032976124091513292491 -0.091578898488961058 0.3865718126789312592 rpy=6.3108872417680804303e-30 -2.9537602700216738211e-30 -3.141592653589793116
- joint liigend_to_kere_joint: origin xyz=0.9483341292917655263 -0.0071774303769965852595 0.6075567520903586427 rpy=2.2686993105948162011e-15 -6.1350116673315255536e-22 -1.5707963267948390484 -> xyz=-0.00017382192779770433422 -0.00024642929502571853106 -0.0034281873210687263676 rpy=0 -0 0
